File: RevA/MidiLedController.sch (KiCad schematic (older format))
At the start: 50 parts, among them J1 Molex 2Way KK254, J12 Barrel_Jack, SW1 SW_DIP_x04, SW2 SW_SPST, U20 STM32F051K8Tx, U21 6N135S

Commit message: updated HW
changed single gang PTD901 to dual gang concentric PTH901
Parts:
- removed RV1: B10K PTD901, Potentiometer_THT:Potentiometer_Bourns_3386C_Horizontal, symbol Device:R_POT
- added C5: 100pF, Capacitor_SMD:C_0805_2012Metric_Pad1.15x1.40mm_HandSolder, symbol Device:C
- added R25: 100R, Resistor_SMD:R_0805_2012Metric_Pad1.15x1.40mm_HandSolder, symbol Device:R
- added RV1: PTH901, PTH901:PTH901, symbol Device:R_POT_Dual_Separate
- added TP3: TestPoint, TestPoint:TestPoint_Pad_1.0x1.0mm, symbol Connector:TestPoint
Connections:
- net +3V3: now also RV1.3, RV1.6
- net ADC_IN1: now also C5.2, R25.2, TP3.1; no longer J_AUX1.2 (Pin_2)
- net ADC_IN2: now also J_AUX1.2 (Pin_2); no longer J_AUX1.1 (Pin_1)
- net GNDS: now also C5.1, RV1.1, RV1.4
- net ADC_IN3: now reaches U20.9 (PA3)
- net ADC_IN3: now also J_AUX1.1 (Pin_1)
- net at R74.1: now also RV1.2
- new net: R25.1, RV1.5
- no-connect marks 10 -> 9
Other:
- moved on the sheet: C26, D2, J_MIDI_IN1, R119, R120, R121, R122, R4, R74, R9, SW1, TP1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
